Commit message: basic control, but still the position is not accurate

File: scripts/niryo_two.urdf (robot description, URDF)
Before this commit: robot niryo_one, 9 links, 8 joints
Links:
- removed link tool_link
- removed link world
- link arm_link: geometry collision mesh filename=package://niryo_one_description/meshes/v2/stl/arm_link.stl; visual mesh filename=package://niryo_one_description/meshes/v2/stl/arm_link.stl
- link base_link: geometry collision mesh filename=package://niryo_one_description/meshes/v2/stl/base_link.stl; visual mesh filename=package://niryo_one_description/meshes/v2/stl/base_link.stl
- link elbow_link: geometry collision mesh filename=package://niryo_one_description/meshes/v2/stl/elbow_link.stl; visual mesh filename=package://niryo_one_description/meshes/v2/stl/elbow_link.stl
- link forearm_link: geometry collision mesh filename=package://niryo_one_description/meshes/v2/stl/forearm_link.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; visual mesh filename=package://niryo_one_description/meshes/v2/stl/forearm_link.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
- link hand_link: geometry collision mesh filename=package://niryo_one_description/meshes/v2/stl/hand_link.stl; visual mesh filename=package://niryo_one_description/meshes/v2/stl/hand_link.stl
- link shoulder_link: geometry collision mesh filename=package://niryo_one_description/meshes/v2/stl/shoulder_link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; visual mesh filename=package://niryo_one_description/meshes/v2/stl/shoulder_link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
- link wrist_link: geometry collision mesh filename=package://niryo_one_description/meshes/v2/stl/wrist_link.stl; visual mesh filename=package://niryo_one_description/meshes/v2/stl/wrist_link.stl
Joints:
- removed joint hand_tool_joint
- removed joint joint_world
- added joint hand_tool_joint_1: type fixed, parent hand_link, child tool_link_1, origin xyz=0.027 0 0.015 rpy=-0.5 0.5 0.5
- added joint hand_tool_joint_2: type fixed, parent hand_link, child tool_link_2, origin xyz=0.027 0 0.015 rpy=-0.5 0.5 0.5
- joint joint_1: limit lower=-3.05433 upper=3.05433 effort=1 velocity=1.0 -> lower=-2.949 upper=2.949 effort=1 velocity=1.0; origin xyz=0 0 0.103 rpy=0 0 0 -> xyz=0 0 0.203 rpy=0 0 0
- joint joint_2: limit lower=-1.57080 upper=0.640187 effort=1 velocity=1.0 -> lower=-1.83 upper=0.61 effort=1 velocity=1.0; origin xyz=0 0 0.080 rpy=1.570796326795 -1.570796326795 0 -> xyz=0 0 0.08 rpy=0.5 -0.5 0
- joint joint_3: limit lower=-1.397485 upper=1.570796326795 effort=1 velocity=1.0 -> lower=-1.34 upper=1.57 effort=1 velocity=1.0; origin xyz=0.210 0.0 0 rpy=0 0 -1.570796326795 -> xyz=0.21 0 0 rpy=0 0 -1.5708
- joint joint_4: limit lower=-3.05433 upper=3.05433 effort=1 velocity=1.0 -> lower=-2.089 upper=2.089 effort=1 velocity=1.0; origin xyz=0.0415 0.030 0 rpy=0 1.570796326795 0 -> xyz=0.0415 0.03 0 rpy=0 1.5708 0
- joint joint_5: origin xyz=0 0 0.180 rpy=0 -1.570796326795 0 -> xyz=0 0 0.18 rpy=0 -1.5708 0
- joint joint_6: origin xyz=0.0164 -0.0055 0 rpy=0 1.570796326795 0 -> xyz=0.0164 -0.0055 0 rpy=0 1.5708 0
