Commit message: control updates, changed the forces, 3D inverse position error

File: scripts/niryo_fixedpos.urdf (robot description, URDF)
Before this commit: robot niryo_one, 10 links, 8 joints
Links:
- removed link tool_link_1
- removed link tool_link_2
- removed link world
- link arm_link: geometry visual mesh filename=package://niryo_one_description/meshes/arm_link.stl
- link base_link: geometry visual mesh filename=package://niryo_one_description/meshes/base_link.stl
- link elbow_link: geometry visual mesh filename=package://niryo_one_description/meshes/elbow_link.stl
- link forearm_link: geometry visual mesh filename=package://niryo_one_description/meshes/forearm_link.stl
- link hand_link: geometry visual mesh filename=package://niryo_one_description/meshes/hand_link.stl
- link shoulder_link: geometry visual mesh filename=package://niryo_one_description/meshes/shoulder_link.stl
- link wrist_link: geometry visual mesh filename=package://niryo_one_description/meshes/wrist_link.stl
Joints:
- removed joint hand_tool_joint_1
- removed joint hand_tool_joint_2
- joint joint_1: limit lower=-2.49433 upper=2.49433 effort=1 velocity=1.0 -> lower=-2.949 upper=2.949 effort=1 velocity=1
- joint joint_2: limit lower=-1.5708 upper=0.640187 effort=1 velocity=1.0 -> lower=-1.83 upper=0.61 effort=2 velocity=1; origin xyz=0 0 0.08 rpy=0.61207963268 -1.3007963268 0 -> xyz=0 0 0.08 rpy=0.5 0.5 -0.5
- joint joint_3: limit lower=-1.34 upper=1.57 effort=1 velocity=1.0 -> lower=-0.51 upper=0.46 effort=2 velocity=1; origin xyz=0.21 0.0 0 rpy=0 0 -1.5707963268 -> xyz=0.21 0 0 rpy=0 0 -0.5708
- joint joint_4: limit lower=-2.089 upper=2.089 effort=1 velocity=1.0 -> lower=-2.089 upper=-0.000 effort=1 velocity=1; origin xyz=0.0415 0.03 0 rpy=0 1.5707963268 0 -> xyz=0.0415 0.03 0 rpy=0 1.5708 0
- joint joint_5: limit lower=-1.74533 upper=1.91986 effort=1 velocity=1.0 -> lower=-1.74533 upper=1.91986 effort=1 velocity=1; origin xyz=0 0 0.18 rpy=0 -1.5707963268 0 -> xyz=0 0 0.19 rpy=0 -1.5708 0
- joint joint_6: limit lower=-2.57436 upper=2.57436 effort=1 velocity=1.0 -> lower=-1.7000 upper=1.5000 effort=1 velocity=1; origin xyz=0.0164 -0.0055 0 rpy=0 1.5707963268 0 -> xyz=0.0164 -0.0055 0 rpy=0 1.5708 0

File: scripts/niryo_robot.urdf (robot description, URDF)
Before this commit: robot niryo_one, 10 links, 8 joints
Joints:
- added joint joint_world: type fixed, parent world, child base_link, origin xyz=0 0 0 rpy=0 0 0
- joint joint_3: limit lower=-1.34 upper=1.57 effort=1 velocity=1.0 -> lower=-0.40 upper=0.07 effort=1 velocity=1.0
- joint joint_5: origin xyz=0 0 0.18 rpy=0 -1.5707963268 0 -> xyz=0 0 0.19 rpy=0 -1.5707963268 0
- joint joint_6: origin xyz=0.0164 -0.0055 0 rpy=0 1.5707963268 0 -> xyz=0.0164 -0.0055 0 rpy=0 0 1.60005; type revolute -> fixed
