Commit message: control almost done, inverse kinematic function is not so correct

File: scripts/niryo_robot.urdf (robot description, URDF)
Before this commit: robot niryo_one, 10 links, 9 joints
Links:
- removed link tool_link_1
- removed link tool_link_2
- added link g1_clamp_left, mass 0.015; collision mesh filename=package://niryo_one_description/meshes/g1_clampLeft.stl; visual mesh filename=package://niryo_one_description/meshes/g1_clampLeft.dae
- added link g1_clamp_right, mass 0.015; collision mesh filename=package://niryo_one_description/meshes/g1_clampRight.stl; visual mesh filename=package://niryo_one_description/meshes/g1_clampRight.dae
- added link g1_main_support, mass 0.04; collision mesh filename=package://niryo_one_tools_support/meshes/gripper_1/stl/g1_m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; visual mesh filename=package://niryo_one_tools_support/meshes/gripper_1/collada/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
Joints:
- removed joint hand_tool_joint_1
- removed joint hand_tool_joint_2
- removed joint joint_world
- added joint ${prefix}niryo_gripper_1_joint: type fixed, parent hand_link, child g1_main_support, origin xyz=0.027 0 0.015  rpy=4.712388980385 0 1.57079632
- added joint left_clamp_joint: type prismatic, parent g1_main_support, child g1_clamp_left, origin xyz=0.027 0 0.015 rpy=0 0 0, axis 1 0 0, limit lower=-0.012 upper=0 effort=100.0 velocity=3.0
- added joint right_clamp_joint: type prismatic, parent g1_main_support, child g1_clamp_right, origin xyz=0.027 0 0.015 rpy=0 0 0, axis 1 0 0, limit lower=0 upper=0.012 effort=100.0 velocity=3.0
- joint joint_3: limit lower=-0.40 upper=0.07 effort=1 velocity=1.0 -> lower=-1.34  upper=1.57 effort=1 velocity=1.0
- joint joint_5: limit lower=-1.74533 upper=1.91986 effort=1 velocity=1.0 -> lower=-1.74533 upper=1.3000 effort=1 velocity=1.0
- joint joint_6: type fixed -> revolute

Commit message: i hate kinematic function. adding a free moving ball but still control is not correct

File: scripts/niryo_robot.urdf (robot description, URDF)
Before this commit: robot niryo_one, 11 links, 9 joints
Joints:
- joint joint_2: limit lower=-1.5708 upper=0.640187 effort=1 velocity=1.0 -> lower=-1.5708 upper=0.61 effort=1 velocity=1.0
- joint joint_4: limit lower=-2.089 upper=2.089 effort=1 velocity=1.0 -> lower=-0.5089 upper=0.5089 effort=1 velocity=1.0
- joint joint_5: limit lower=-1.74533 upper=1.3000 effort=1 velocity=1.0 -> lower=-0.2397 upper=0.2397 effort=1 velocity=1.0
- joint left_clamp_joint: limit lower=-0.012 upper=0 effort=100.0 velocity=3.0 -> lower=-0.0120000 upper=0 effort=100.0 velocity=3.0
- joint right_clamp_joint: limit lower=0 upper=0.012 effort=100.0 velocity=3.0 -> lower=0 upper=0.0120000 effort=100.0 velocity=3.0

Commit message: DON'T CHANGE THE MODEL AGAIN!! FINAL VERSION OF THE HARDWARE PART

File: scripts/niryo_robot.urdf (robot description, URDF)
Before this commit: robot niryo_one, 11 links, 9 joints
Joints:
- joint joint_5: limit lower=-0.2397 upper=0.2397 effort=1 velocity=1.0 -> lower=-0.02397 upper=0.02397 effort=1 velocity=1.0
